File: .github/tests/test pcb/test.kicad_pcb (KiCad board)
At the start: 2 copper layers, 2 parts

Commit message: Add more tests
Other:
- board text added: "Front ███"
- board text removed: "Front"
Changed lines of the file:
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@@
 		)
 	)
-	(gr_text "Front"
+	(gr_text "Front ███"
 		(at 177.5 98 0)
 		(layer "F.SilkS")
 		(effects
 			(font
+			    (face "Arial")
 				(size 1 1)
 				(thickness 0.1)
